Commit message: add gazebo camera plugin

File: catkin_ws/src/simulation/husky_description/urdf/husky_walker.urdf.xacro (robot description, xacro)
@@ -22,7 +22,10 @@
 -->
 <robot name="husky" xmlns:xacro="http://ros.org/wiki/xacro">
-  <xacro:arg name="laser_enabled" default="false" />
-  <xacro:arg name="laser_xyz" default="$(optenv HUSKY_LMS1XX_XYZ 0.2206 0.0 0.00635)" />
-  <xacro:arg name="laser_rpy" default="$(optenv HUSKY_LMS1XX_RPY 0.0 0.0 0.0)" />
+  <xacro:arg name="ydlidar_enabled" default="true" />
+  <xacro:arg name="ydlidar_xyz" default="$(optenv HUSKY_YDLIDAR_XYZ 0.41 0.0 0.535)" />
+  <xacro:arg name="ydlidar_rpy" default="$(optenv HUSKY_YDLIDAR_RPY 0.0 0.0 3.1415926)" />
+  <xacro:arg name="webcam_enabled" default="true" />
+  <xacro:arg name="webcam_xyz" default="$(optenv HUSKY_WEBCAM_XYZ -4.0e-02 0 -3.25e-02)" />
+  <xacro:arg name="webcam_rpy" default="$(optenv HUSKY_WEBCAM_RPY 0 0 3.1415926)" />
   <xacro:arg name="realsense_enabled" default="false" />
   <xacro:arg name="realsense_xyz" default="$(optenv HUSKY_REALSENSE_XYZ 0 0 0)" />
@@ -37,6 +40,7 @@
   <xacro:include filename="$(find husky_description)/urdf/wheel.urdf.xacro" />
   <xacro:include filename="$(find husky_description)/urdf/accessories/intel_realsense.urdf.xacro"/>
-  <xacro:include filename="$(find husky_description)/urdf/accessories/sick_lms1xx_mount.urdf.xacro"/>
+  <xacro:include filename="$(find husky_description)/urdf/accessories/webcam_c930e.urdf.xacro"/>
   <xacro:include filename="$(find husky_description)/urdf/accessories/sensor_arch.urdf.xacro"/>
+  <xacro:include filename="$(find ydlidar)/urdf/ydlidar_g4.urdf.xacro" />
   <xacro:property name="M_PI" value="3.14159"/>
   <!-- Base Size -->
@@ -116,20 +120,20 @@
   </xacro:husky_wheel>
   <xacro:husky_decorate />
-  <xacro:if value="$(arg laser_enabled)">
-    <sick_lms1xx_mount prefix="base"/>
-    <sick_lms1xx frame="base_laser" topic="scan" robot_namespace="$(arg robot_namespace)"/>
-    <joint name="laser_mount_joint" type="fixed">
-      <origin xyz="$(arg laser_xyz)" rpy="$(arg laser_rpy)" />
-      <parent link="top_plate_link" />
-      <child link="base_laser_mount" />
+  <xacro:if value="$(arg ydlidar_enabled)">
+    <ydlidar_g4 frame="laser" topic="scan" robot_namespace="$(arg robot_namespace)"/>
+    <joint name="ydlidar_mount_joint" type="fixed">
+        <origin xyz="$(arg ydlidar_xyz)" rpy="$(arg ydlidar_rpy)" />
+        <parent link="base_link" />
+        <child link="laser_base" />
     </joint>
   </xacro:if>
-  <!-- <xacro:include filename="$(find ydlidar)/urdf/ydlidar_g4.urdf.xacro" />
-    <ydlidar_g4 name="ydlidar_g4_v0" ros_topic="scan2" />
-    <joint name="ydlidar_mount_joint" type="fixed">
-      <origin xyz="0.2206 0.0 0.40635" rpy="$(arg laser_rpy)" />
-      <parent link="top_plate_link" />
-      <child link="ydlidar_g4_v0_base" />
-  </joint> -->
+  <xacro:if value="$(arg webcam_enabled)">
+    <webcam_c930e frame="camera" topic="usb_cam" robot_namespace="$(arg robot_namespace)"/>
+    <joint name="webcam_mount_joint" type="fixed">
+        <origin xyz="$(arg webcam_xyz)" rpy="$(arg webcam_rpy)" />
+        <parent link="laser_link" />
+        <child link="camera_link" />
+    </joint>
+  </xacro:if>
   <!--
     top sensor arch; include this if we have realsense enabled
