Commit message: add pedsim_ros

File: catkin_ws/src/simulation/walker_description/urdf/accessories/webcam_c930e.urdf.xacro (robot description, xacro)
@@ -62,5 +62,5 @@
                     <imageTopicName>image_raw</imageTopicName>
                     <cameraInfoTopicName>camera_info</cameraInfoTopicName>
-                    <frameName>${frame}_optical_frame</frameName>
+                    <frameName>/${frame}_optical_frame</frameName>
                     <hackBaseline>0.07</hackBaseline>
                     <distortionK1>0.00000001</distortionK1>
@@ -73,4 +73,5 @@
                     <Cy>0</Cy>
                     <focalLength>0</focalLength>
+                    <robotNamespace>$(arg robot_namespace)</robotNamespace>
                 </plugin>
             </sensor>

File: catkin_ws/src/simulation/walker_description/urdf/walker.urdf.xacro (robot description, xacro)
@@ -203,5 +203,6 @@
             <origin xyz="0 0 0" rpy="0 0 0" />
             <geometry>
-                <mesh filename="package://walker_description/meshes/front_caster_wheel_link.STL" />
+                <!-- <mesh filename="package://walker_description/meshes/front_caster_wheel_link.STL" /> -->
+                <sphere radius="${front_wheel_radius + 0.03}"/>
             </geometry>
             <material name="">
@@ -212,5 +213,6 @@
             <origin xyz="0 0 0" rpy="0 0 0" />
             <geometry>
-                <mesh filename="package://walker_description/meshes/front_caster_wheel_link.STL" />
+                <!-- <mesh filename="package://walker_description/meshes/front_caster_wheel_link.STL" /> -->
+                <sphere radius="${front_wheel_radius + 0.03}"/>
             </geometry>
         </collision>
@@ -232,5 +234,6 @@
             <origin xyz="0 0 0" rpy="0 0 0" />
             <geometry>
-                <mesh filename="package://walker_description/meshes/front_caster_wheel_link.STL" />
+                <!-- <mesh filename="package://walker_description/meshes/front_caster_wheel_link.STL" /> -->
+                <sphere radius="${front_wheel_radius + 0.03}"/>
             </geometry>
             <material name="">
@@ -241,5 +244,6 @@
             <origin xyz="0 0 0" rpy="0 0 0" />
             <geometry>
-                <mesh filename="package://walker_description/meshes/front_caster_wheel_link.STL" />
+                <!-- <mesh filename="package://walker_description/meshes/front_caster_wheel_link.STL" /> -->
+                <sphere radius="${front_wheel_radius + 0.03}"/>
             </geometry>
         </collision>
