Commit message: fix robot model problem

File: catkin_ws/src/simulation/walker_description/urdf/walker.urdf.xacro (robot description, xacro)
@@ -4,4 +4,9 @@
     <xacro:arg name="laser_xyz" default="$(optenv HUSKY_LMS1XX_XYZ 0.2206 0.0 0.00635)" />
     <xacro:arg name="laser_rpy" default="$(optenv HUSKY_LMS1XX_RPY 0.0 0.0 0.0)" />
+    <xacro:arg name="rear_wheel_mass" default="1.0" />
+    <xacro:arg name="rear_wheel_radius" default="0.0625" />
+    <xacro:arg name="rear_wheel_width" default="0.02" />
+    <xacro:arg name="front_wheel_mass" default="0.5" />
+    <xacro:arg name="front_wheel_radius" default="0.025" />
     <!-- <xacro:arg name="robot_namespace" default="/" />  -->
     <xacro:arg name="robot_namespace" default="active_walker" />
@@ -17,5 +22,5 @@
     <link name="base_link">
         <inertial>
-            <origin xyz="0.26321 1.2785E-06 0.15671" rpy="0 0 0" />
+            <origin xyz="0.26321 0.0 0.15671" rpy="0 0 0" />
             <!-- <mass value="3.5774" /> -->
             <mass value="7.0" />
@@ -43,14 +48,14 @@
         <inertial>
             <origin xyz="0 0 0" rpy="0 0 0" />
-            <!-- <mass value="0.18877" /> -->
-            <mass value="10.0" />
+            <mass value="$(arg rear_wheel_mass)" />
             <!-- <inertia ixx="0.00013887" ixy="-1.6386E-36" ixz="2.1452E-37"
                     iyy="0.00013887" iyz="-7.5427E-20" izz="0.00026251" /> -->
-            <cylinder_inertia m="10.0" r="0.0625" h="0.02" />
-        </inertial>
-        <visual>
-            <origin xyz="0 0 0" rpy="0 0 0" />
-            <geometry>
-                <mesh filename="package://walker_description/meshes/rear_right_wheel_link.STL" />
+            <cylinder_inertia m="$(arg rear_wheel_mass)" r="$(arg rear_wheel_radius)" h="$(arg rear_wheel_width)" />
+        </inertial>
+        <visual>
+            <origin xyz="0 0 0" rpy="0 0 0" />
+            <geometry>
+                <!-- <mesh filename="package://walker_description/meshes/rear_right_wheel_link.STL" /> -->
+                <cylinder length="$(arg rear_wheel_width)" radius="$(arg rear_wheel_radius)"/>
             </geometry>
             <material name="">
@@ -61,5 +66,6 @@
             <origin xyz="0 0 0" rpy="0 0 0" />
             <geometry>
-                <mesh filename="package://walker_description/meshes/rear_right_wheel_link.STL" />
+                <!-- <mesh filename="package://walker_description/meshes/rear_right_wheel_link.STL" /> -->
+                <cylinder length="$(arg rear_wheel_width)" radius="$(arg rear_wheel_radius)"/>
             </geometry>
         </collision>
@@ -69,6 +75,9 @@
         <parent link="base_link" />
         <child link="rear_right_wheel_link" />
-        <axis xyz="0 0.099176 0.99507" />
-        <dynamics friction="0.001" />
+        <!-- <axis xyz="0 0.099176 0.99507" /> -->
+        <axis xyz="0 0 1" />
+        <!-- <dynamics friction="0.001" /> -->
+        <joint_properties damping="0.0" friction="0.0"/>
+        <limit effort="100" velocity="100"/>
     </joint>
     <!-- Rear left wheel link & joint -->
@@ -76,14 +85,14 @@
         <inertial>
             <origin xyz="0 0 0" rpy="0 0 0" />
-            <!-- <mass value="0.18877" /> -->
-            <mass value="10.0" />
+            <mass value="$(arg rear_wheel_mass)" />
             <!-- <inertia ixx="0.00013887" ixy="4.2884E-36" ixz="-8.5028E-20"
                     iyy="0.00013887" iyz="-7.5708E-21" izz="0.00026251" /> -->
-            <cylinder_inertia m="10.0" r="0.0625" h="0.02" />
-        </inertial>
-        <visual>
-            <origin xyz="0 0 0" rpy="0 0 0" />
-            <geometry>
-                <mesh filename="package://walker_description/meshes/rear_left_wheel_link.STL" />
+            <cylinder_inertia m="$(arg rear_wheel_mass)" r="$(arg rear_wheel_radius)" h="$(arg rear_wheel_width)" />
+        </inertial>
+        <visual>
+            <origin xyz="0 0 0" rpy="0 0 0" />
+            <geometry>
+                <!-- <mesh filename="package://walker_description/meshes/rear_left_wheel_link.STL" /> -->
+                <cylinder length="$(arg rear_wheel_width)" radius="$(arg rear_wheel_radius)"/>
             </geometry>
             <material name="">
@@ -94,5 +103,6 @@
             <origin xyz="0 0 0" rpy="0 0 0" />
             <geometry>
-                <mesh filename="package://walker_description/meshes/rear_left_wheel_link.STL" />
+                <!-- <mesh filename="package://walker_description/meshes/rear_left_wheel_link.STL" /> -->
+                <cylinder length="$(arg rear_wheel_width)" radius="$(arg rear_wheel_radius)"/>
             </geometry>
         </collision>
@@ -102,7 +112,10 @@
         <parent link="base_link" />
         <child link="rear_left_wheel_link" />
-        <axis xyz="0 0.099176 0.99507" />
-        <limit lower="0" upper="0" effort="0" velocity="0" />
-        <dynamics friction="0.001" />
+        <!-- <axis xyz="0 0.099176 0.99507" /> -->
+        <axis xyz="0 0 1" />
+        <!-- <limit lower="0" upper="0" effort="0" velocity="0" /> -->
+        <!-- <dynamics friction="0.001" /> -->
+        <joint_properties damping="0.0" friction="0.0"/>
+        <limit effort="100" velocity="100"/>
     </joint>
     <!-- Force sensor link & joint -->
@@ -171,10 +184,7 @@
     <link name="front_right_caster_wheel_link">
         <inertial>
-            <origin xyz="-0.0042994 2.0823E-06 -0.0092241" rpy="0 0 0" />
-            <!-- <mass value="0.062864" /> -->
-            <mass value="0.5" />
-            <!-- <inertia ixx="1.8333E-05" ixy="-2.766E-10" ixz="-4.2964E-07"
-                    iyy="3.1598E-05" iyz="-9.745E-11" izz="2.0211E-05" /> -->
-            <sphere_inertia m="0.5" r="0.025"/>
+            <origin xyz="0 0 0" rpy="0 0 0" />
+            <mass value="$(arg front_wheel_mass)" />
+            <sphere_inertia m="$(arg front_wheel_mass)" r="$(arg front_wheel_radius)"/>
         </inertial>
         <visual>
@@ -203,10 +213,7 @@
     <link name="front_left_caster_wheel_link">
         <inertial>
-            <origin xyz="-0.0042994 2.0823E-06 -0.0092241" rpy="0 0 0" />
-            <!-- <mass value="0.062864" /> -->
-            <mass value="0.5" />
-            <!-- <inertia ixx="1.8333E-05" ixy="-2.766E-10" ixz="-4.2964E-07"
-                    iyy="3.1598E-05" iyz="-9.745E-11" izz="2.0211E-05" /> -->
-            <sphere_inertia m="0.5" r="0.025"/>
+            <origin xyz="0 0 0" rpy="0 0 0" />
+            <mass value="$(arg front_wheel_mass)" />
+            <sphere_inertia m="$(arg front_wheel_mass)" r="$(arg front_wheel_radius)"/>
         </inertial>
         <visual>

Commit message: fix simulation tf bug

File: catkin_ws/src/simulation/walker_description/urdf/walker.urdf.xacro (robot description, xacro)
@@ -44,4 +44,11 @@
         </collision>
     </link>
+    <!-- Footprint -->
+    <!-- <link name="footprint" />
+    <joint name="footprint_joint" type="fixed">
+        <origin xyz="0 0 -0.12671" rpy="0 0 0" />
+        <parent link="base_link"/>
+        <child link="footprint"/>
+    </joint> -->
     <!-- Rear right wheel link & joint -->
     <link name="rear_right_wheel_link">

Commit message: fix tf not working problem

File: catkin_ws/src/simulation/walker_description/urdf/walker.urdf.xacro (robot description, xacro)
@@ -1,17 +1,9 @@
 <?xml version="1.0" encoding="UTF-8"?>
 <robot name="active_walker" xmlns:xacro="http://ros.org/wiki/xacro">
-    <xacro:arg name="laser_enabled" default="false" />
-    <xacro:arg name="laser_xyz" default="$(optenv HUSKY_LMS1XX_XYZ 0.2206 0.0 0.00635)" />
-    <xacro:arg name="laser_rpy" default="$(optenv HUSKY_LMS1XX_RPY 0.0 0.0 0.0)" />
-    <xacro:arg name="rear_wheel_mass" default="1.0" />
-    <xacro:arg name="rear_wheel_radius" default="0.0625" />
-    <xacro:arg name="rear_wheel_width" default="0.02" />
-    <xacro:arg name="front_wheel_mass" default="0.5" />
-    <xacro:arg name="front_wheel_radius" default="0.025" />
     <!-- <xacro:arg name="robot_namespace" default="/" />  -->
     <xacro:arg name="robot_namespace" default="active_walker" />
     <!-- Included URDF/XACRO Files -->
-    <!-- <xacro:include filename="$(find husky_description)/urdf/accessories/webcam_c930e.urdf.xacro"/> -->
-    <!-- <xacro:include filename="$(find ydlidar)/urdf/ydlidar_g4.urdf.xacro" /> -->
+    <xacro:include filename="$(find walker_description)/urdf/accessories/webcam_c930e.urdf.xacro"/>
+    <xacro:include filename="$(find walker_description)/urdf/accessories/ydlidar_g4.urdf.xacro" />
     <!-- Gazebo plugin -->
     <xacro:include filename="$(find walker_description)/urdf/walker.gazebo" />
@@ -19,4 +11,13 @@
     <xacro:include filename="$(find walker_description)/urdf/macros.xacro" />
     <xacro:property name="M_PI" value="3.1415926"/>
+    <xacro:property name="rear_wheel_mass" value="1.0" />
+    <xacro:property name="rear_wheel_radius" value="0.0625" />
+    <xacro:property name="rear_wheel_width" value="0.02" />
+    <xacro:property name="front_wheel_mass" value="0.5" />
+    <xacro:property name="front_wheel_radius" value="0.025" />
+    <xacro:property name="ydlidar_xyz" value="$(optenv HUSKY_YDLIDAR_XYZ 0.41 0.0 0.535)" />
+    <xacro:property name="ydlidar_rpy" value="$(optenv HUSKY_YDLIDAR_RPY 0.0 0.0 3.1415926)" />
+    <xacro:property name="webcam_xyz" value="$(optenv HUSKY_WEBCAM_XYZ -4.0e-02 0 -3.25e-02)" />
+    <xacro:property name="webcam_rpy" value="$(optenv HUSKY_WEBCAM_RPY 0 0 3.1415926)" />
     <!-- Base link -->
     <link name="base_link">
@@ -55,8 +56,8 @@
         <inertial>
             <origin xyz="0 0 0" rpy="0 0 0" />
-            <mass value="$(arg rear_wheel_mass)" />
+            <mass value="${rear_wheel_mass}" />
             <!-- <inertia ixx="0.00013887" ixy="-1.6386E-36" ixz="2.1452E-37"
                     iyy="0.00013887" iyz="-7.5427E-20" izz="0.00026251" /> -->
-            <cylinder_inertia m="$(arg rear_wheel_mass)" r="$(arg rear_wheel_radius)" h="$(arg rear_wheel_width)" />
+            <cylinder_inertia m="${rear_wheel_mass}" r="${rear_wheel_radius}" h="${rear_wheel_width}" />
         </inertial>
         <visual>
@@ -64,5 +65,5 @@
             <geometry>
                 <!-- <mesh filename="package://walker_description/meshes/rear_right_wheel_link.STL" /> -->
-                <cylinder length="$(arg rear_wheel_width)" radius="$(arg rear_wheel_radius)"/>
+                <cylinder length="${rear_wheel_width}" radius="${rear_wheel_radius}"/>
             </geometry>
             <material name="">
@@ -74,5 +75,5 @@
             <geometry>
                 <!-- <mesh filename="package://walker_description/meshes/rear_right_wheel_link.STL" /> -->
-                <cylinder length="$(arg rear_wheel_width)" radius="$(arg rear_wheel_radius)"/>
+                <cylinder length="${rear_wheel_width}" radius="${rear_wheel_radius}"/>
             </geometry>
         </collision>
@@ -92,8 +93,8 @@
         <inertial>
             <origin xyz="0 0 0" rpy="0 0 0" />
-            <mass value="$(arg rear_wheel_mass)" />
+            <mass value="${rear_wheel_mass}" />
             <!-- <inertia ixx="0.00013887" ixy="4.2884E-36" ixz="-8.5028E-20"
                     iyy="0.00013887" iyz="-7.5708E-21" izz="0.00026251" /> -->
-            <cylinder_inertia m="$(arg rear_wheel_mass)" r="$(arg rear_wheel_radius)" h="$(arg rear_wheel_width)" />
+            <cylinder_inertia m="${rear_wheel_mass}" r="${rear_wheel_radius}" h="${rear_wheel_width}" />
         </inertial>
         <visual>
@@ -101,5 +102,5 @@
             <geometry>
                 <!-- <mesh filename="package://walker_description/meshes/rear_left_wheel_link.STL" /> -->
-                <cylinder length="$(arg rear_wheel_width)" radius="$(arg rear_wheel_radius)"/>
+                <cylinder length="${rear_wheel_width}" radius="${rear_wheel_radius}"/>
             </geometry>
             <material name="">
@@ -111,5 +112,5 @@
             <geometry>
                 <!-- <mesh filename="package://walker_description/meshes/rear_left_wheel_link.STL" /> -->
-                <cylinder length="$(arg rear_wheel_width)" radius="$(arg rear_wheel_radius)"/>
+                <cylinder length="${rear_wheel_width}" radius="${rear_wheel_radius}"/>
             </geometry>
         </collision>
@@ -128,32 +129,36 @@
     <!-- Force sensor link & joint -->
     <link name="force_sensor_link">
-    <inertial>
-        <origin xyz="0.0041884 0.0015924 0.015541" rpy="0 0 0" />
-        <!-- <mass value="0.17912" /> -->
-        <mass value="0.5" />
-        <inertia ixx="8.7156E-05" ixy="-9.4168E-06" ixz="4.2663E-06"
-                iyy="0.00011084" iyz="1.6414E-06" izz="0.0001673" />
-    </inertial>
-    <visual>
-        <origin xyz="0 0 0" rpy="0 0 0" />
-        <geometry>
-            <mesh filename="package://walker_description/meshes/force_sensor_link.STL" />
-        </geometry>
-        <material name="">
-            <color rgba="0.9569 0.2196 0 1" />
-        </material>
-    </visual>
-    <collision>
-        <origin xyz="0 0 0" rpy="0 0 0" />
-        <geometry>
-            <mesh filename="package://walker_description/meshes/force_sensor_link.STL" />
-        </geometry>
-    </collision>
-    </link>
-    <joint name="force_sensor_joint" type="fixed">
+        <inertial>
+            <origin xyz="0.0041884 0.0015924 0.015541" rpy="0 0 0" />
+            <!-- <mass value="0.17912" /> -->
+            <mass value="0.5" />
+            <!-- <inertia ixx="8.7156E-05" ixy="-9.4168E-06" ixz="4.2663E-06"
+                    iyy="0.00011084" iyz="1.6414E-06" izz="0.0001673" /> -->
+            <cylinder_inertia m="0.5" r="0.04" h="0.03" />
+        </inertial>
+        <visual>
+            <origin xyz="0 0 0" rpy="0 0 0" />
+            <geometry>
+                <mesh filename="package://walker_description/meshes/force_sensor_link.STL" />
+            </geometry>
+            <material name="">
+                <color rgba="0.9569 0.2196 0 1" />
+            </material>
+        </visual>
+        <collision>
+            <origin xyz="0 0 0" rpy="0 0 0" />
+            <geometry>
+                <mesh filename="package://walker_description/meshes/force_sensor_link.STL" />
+            </geometry>
+        </collision>
+    </link>
+    <joint name="force_sensor_joint" type="revolute"> <!-- fixed -->
         <origin xyz="0.16109 0 0.81585" rpy="0 0 -1.5708" />
         <parent link="base_link" />
         <child link="force_sensor_link" />
-        <axis xyz="0 0 0" />
+        <axis xyz="0 0 1" />
+        <limit lower="0" velocity="1000" upper="0" effort="1000" />
+        <!-- <safety_controller k_velocity="10" k_position="15" soft_lower_limit="-2.0" soft_upper_limit="0.5" />
+        <dynamics damping="0.0" friction="0.0"/> -->
     </joint>
     <!-- Handrail link -->
@@ -192,11 +197,11 @@
         <inertial>
             <origin xyz="0 0 0" rpy="0 0 0" />
-            <mass value="$(arg front_wheel_mass)" />
-            <sphere_inertia m="$(arg front_wheel_mass)" r="$(arg front_wheel_radius)"/>
-        </inertial>
-        <visual>
-            <origin xyz="0 0 0" rpy="0 0 0" />
-            <geometry>
-                <mesh filename="package://walker_description/meshes/front_right_caster_wheel_link.STL" />
+            <mass value="${front_wheel_mass}" />
+            <sphere_inertia m="${front_wheel_mass}" r="${front_wheel_radius}"/>
+        </inertial>
+        <visual>
+            <origin xyz="0 0 0" rpy="0 0 0" />
+            <geometry>
+                <mesh filename="package://walker_description/meshes/front_caster_wheel_link.STL" />
             </geometry>
             <material name="">
@@ -207,5 +212,5 @@
             <origin xyz="0 0 0" rpy="0 0 0" />
             <geometry>
-                <mesh filename="package://walker_description/meshes/front_right_caster_wheel_link.STL" />
+                <mesh filename="package://walker_description/meshes/front_caster_wheel_link.STL" />
             </geometry>
         </collision>
@@ -221,11 +226,11 @@
         <inertial>
             <origin xyz="0 0 0" rpy="0 0 0" />
-            <mass value="$(arg front_wheel_mass)" />
-            <sphere_inertia m="$(arg front_wheel_mass)" r="$(arg front_wheel_radius)"/>
-        </inertial>
-        <visual>
-            <origin xyz="0 0 0" rpy="0 0 0" />
-            <geometry>
-                <mesh filename="package://walker_description/meshes/front_left_caster_wheel_link.STL" />
+            <mass value="${front_wheel_mass}" />
+            <sphere_inertia m="${front_wheel_mass}" r="${front_wheel_radius}"/>
+        </inertial>
+        <visual>
+            <origin xyz="0 0 0" rpy="0 0 0" />
+            <geometry>
+                <mesh filename="package://walker_description/meshes/front_caster_wheel_link.STL" />
             </geometry>
             <material name="">
@@ -236,5 +241,5 @@
             <origin xyz="0 0 0" rpy="0 0 0" />
             <geometry>
-                <mesh filename="package://walker_description/meshes/front_left_caster_wheel_link.STL" />
+                <mesh filename="package://walker_description/meshes/front_caster_wheel_link.STL" />
             </geometry>
         </collision>
@@ -246,3 +251,17 @@
         <axis xyz="0 0 0" />
     </joint>
+    <!-- YDLiDAR G4 plugin -->
+    <ydlidar_g4 frame="laser" topic="scan" robot_namespace="$(arg robot_namespace)"/>
+    <joint name="ydlidar_mount_joint" type="fixed">
+        <origin xyz="${ydlidar_xyz}" rpy="${ydlidar_rpy}" />
+        <parent link="base_link" />
+        <child link="laser_base" />
+    </joint>
+    <!-- Logitech C930e webcam -->
+    <webcam_c930e frame="camera" topic="usb_cam" robot_namespace="$(arg robot_namespace)"/>
+    <joint name="webcam_mount_joint" type="fixed">
+        <origin xyz="${webcam_xyz}" rpy="${webcam_rpy}" />
+        <parent link="laser_link" />
+        <child link="camera_link" />
+    </joint>
 </robot>

Commit message: fix robot-regardless bug of simulated pedestrian

File: catkin_ws/src/simulation/walker_description/urdf/walker.urdf.xacro (robot description, xacro)
@@ -52,4 +52,10 @@
         <child link="footprint"/>
     </joint> -->
+    <link name="base_footprint" />
+    <joint name="footprint_joint" type="fixed">
+        <origin xyz="0 0 -0.15671" rpy="0 0 0" />
+        <parent link="base_link"/>
+        <child link="base_footprint"/>
+    </joint>
     <!-- Rear right wheel link & joint -->
     <link name="rear_right_wheel_link">
